File: ODriveInterfacingBoard/ODriveInterfacingBoard.kicad_pcb (KiCad board)
At the start: 2 copper layers, 144.3 x 81.3 mm, 1 part

Commit message: finished footprints started layout
Parts:
- added 50W2RJ1: 50W2RJ1, Footprints:PowerResistorMounts, F.Cu at (259.4, 132.5)
- added Conn1: Molex_SL_02, MRDT_Connectors:MOLEX_SL_02_Horizontal, F.Cu at (224.8, 32.5)
- added Conn13: Molex_SL_09, MRDT_Connectors:MOLEX_SL_09_Horizontal, F.Cu at (160.0, 28.7)
- added Conn14: Molex_SL_05, MRDT_Connectors:MOLEX_SL_05_Horizontal, F.Cu at (182.4, 28.7)
- added Conn2: Molex_SL_05, MRDT_Connectors:MOLEX_SL_05_Horizontal, F.Cu at (137.7, 28.7)
- added Conn3: AndersonPP, MRDT_Connectors:Anderson_2_Horizontal_Side_by_Side, F.Cu at (96.7, 34.7)
- added Conn4: Molex_SL_07, MRDT_Connectors:MOLEX_SL_07_Horizontal, F.Cu at (224.8, 28.7)
- added Conn5: Molex_SL_07, MRDT_Connectors:MOLEX_SL_07_Horizontal, F.Cu at (202.2, 28.7)
- added Conn6: Molex_SL_07, MRDT_Connectors:MOLEX_SL_07_Horizontal, F.Cu at (130.8, -16.8)
- added Conn7: M0_A, MRDT_Connectors:Anderson_3_Horizontal_Side_by_Side, F.Cu at (237.2, 39.2)
- added Conn8: M1_A, MRDT_Connectors:Anderson_3_Horizontal_Side_by_Side, F.Cu at (96.8, 61.6)
- added D1: Tx Yellow, LED_SMD:LED_0603_1608Metric_Pad1.05x0.95mm_HandSolder, F.Cu at (266.8, 158.3)
- added D10: M0 B High Orange, LED_SMD:LED_0603_1608Metric_Pad1.05x0.95mm_HandSolder, F.Cu at (330.5, 133.5)
- added D11: M1 C High Orange, LED_SMD:LED_0603_1608Metric_Pad1.05x0.95mm_HandSolder, F.Cu at (283.8, 156.7)
- added D12: M0 B Low Orange, LED_SMD:LED_0603_1608Metric_Pad1.05x0.95mm_HandSolder, F.Cu at (270.2, 156.7)
- added D13: M1 C Low Orange, LED_SMD:LED_0603_1608Metric_Pad1.05x0.95mm_HandSolder, F.Cu at (273.6, 156.7)
- added D14: M0 C High Orange, LED_SMD:LED_0603_1608Metric_Pad1.05x0.95mm_HandSolder, F.Cu at (277.0, 156.7)
- added D15: M0 C Low Orange, LED_SMD:LED_0603_1608Metric_Pad1.05x0.95mm_HandSolder, F.Cu at (280.4, 156.7)
- added D2: Rx Yellow, LED_SMD:LED_0603_1608Metric_Pad1.05x0.95mm_HandSolder, F.Cu at (400.9, 78.0)
- added D3: M1 A High Orange, LED_SMD:LED_0603_1608Metric_Pad1.05x0.95mm_HandSolder, F.Cu at (320.0, 148.1)
- added D4: 3v3 Green, LED_SMD:LED_0603_1608Metric_Pad1.05x0.95mm_HandSolder, F.Cu at (260.0, 156.7)
- added D5: M1 A Low Orange, LED_SMD:LED_0603_1608Metric_Pad1.05x0.95mm_HandSolder, F.Cu at (303.5, 142.1)
- added D6: M0 A High Orange, LED_SMD:LED_0603_1608Metric_Pad1.05x0.95mm_HandSolder, F.Cu at (263.4, 156.7)
- added D7: M1 B High Orange, LED_SMD:LED_0603_1608Metric_Pad1.05x0.95mm_HandSolder, F.Cu at (260.0, 158.3)
- added D8: M0 A Low Orange, LED_SMD:LED_0603_1608Metric_Pad1.05x0.95mm_HandSolder, F.Cu at (266.8, 156.7)
- added D9: M1 B Low Orange, LED_SMD:LED_0603_1608Metric_Pad1.05x0.95mm_HandSolder, F.Cu at (263.4, 158.3)
- added R1: 1.5k, Resistor_SMD:R_0603_1608Metric_Pad1.05x0.95mm_HandSolder, F.Cu at (290.5, 156.6)
- added R10: 1.5k, Resistor_SMD:R_0603_1608Metric_Pad1.05x0.95mm_HandSolder, F.Cu at (303.5, 143.6)
- added R11: 1.5k, Resistor_SMD:R_0603_1608Metric_Pad1.05x0.95mm_HandSolder, F.Cu at (303.5, 145.1)
- added R12: 1.5k, Resistor_SMD:R_0603_1608Metric_Pad1.05x0.95mm_HandSolder, F.Cu at (293.8, 157.5)
- added R13: 1.5k, Resistor_SMD:R_0603_1608Metric_Pad1.05x0.95mm_HandSolder, F.Cu at (297.2, 156.6)
- added R14: 1.5k, Resistor_SMD:R_0603_1608Metric_Pad1.05x0.95mm_HandSolder, F.Cu at (300.5, 156.6)
- added R15: 1.5k, Resistor_SMD:R_0603_1608Metric_Pad1.05x0.95mm_HandSolder, F.Cu at (303.9, 156.6)
- added R2: 1.5k, Resistor_SMD:R_0603_1608Metric_Pad1.05x0.95mm_HandSolder, F.Cu at (287.1, 158.1)
- added R3: 1.5k, Resistor_SMD:R_0603_1608Metric_Pad1.05x0.95mm_HandSolder, F.Cu at (290.5, 158.1)
- added R4: 1.5k, Resistor_SMD:R_0603_1608Metric_Pad1.05x0.95mm_HandSolder, F.Cu at (270.2, 158.2)
- added R5: 1.5k, Resistor_SMD:R_0603_1608Metric_Pad1.05x0.95mm_HandSolder, F.Cu at (273.5, 158.2)
- added R6: 1.5k, Resistor_SMD:R_0603_1608Metric_Pad1.05x0.95mm_HandSolder, F.Cu at (287.1, 156.6)
- added R7: 1.5k, Resistor_SMD:R_0603_1608Metric_Pad1.05x0.95mm_HandSolder, F.Cu at (276.9, 158.2)
- added R8: 1.5k, Resistor_SMD:R_0603_1608Metric_Pad1.05x0.95mm_HandSolder, F.Cu at (280.2, 158.2)
- added R9: 1.5k, Resistor_SMD:R_0603_1608Metric_Pad1.05x0.95mm_HandSolder, F.Cu at (283.6, 158.2)
- added U1: ODrive, Footprints:ODriveInterfacingBoard, F.Cu at (96.8, 116.8)
Other:
- board size 144.3 x 81.3 mm -> 144.3 x 127.8 mm

Commit message: high level layout
Parts:
- moved D3 285.8 mm to (48.6, 58.4)
- moved D2 285.2 mm to (115.7, 82.3)
- moved D5 267.3 mm to (48.6, 61.5)
- moved D11 248.0 mm to (50.7, 72.1)
- moved D13 236.9 mm to (50.8, 76.2), turned to 180 degrees
- moved D9 232.5 mm to (49.1, 68.1)
- moved D7 231.4 mm to (48.3, 65.0)
- moved D1 207.4 mm to (75.0, 79.2)
- moved D4 190.9 mm to (84.5, 81.8)
- moved 50W2RJ1 185.8 mm to (78.2, 91.4)
- moved R10 182.4 mm to (124.5, 108.7)
- moved R7 180.3 mm to (99.4, 126.5)
- moved R4 178.9 mm to (95.0, 121.9)
- moved R8 176.4 mm to (107.6, 121.9)
- moved R15 175.4 mm to (130.9, 127.5)
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Connections:
- 50W2RJ1 pad 2: Net-(50W2RJ1-Pad2) -> Net-(50W2RJ1-Pad1)
- Conn3 pad 2: (no net) -> PV+
- U1 pad 1: (no net) -> M0_A
Routing:
- net M1_A: track 0.00 -> 101.1 mm
- net M1_B: track 0.00 -> 89.3 mm
- net M0_C: track 0.00 -> 81.2 mm
- net Net-(50W2RJ1-Pad1): track 0.00 -> 81.2 mm
- net M1_C: track 0.00 -> 77.4 mm
- net Net-(50W2RJ1-Pad2): track 0.00 -> 73.6 mm
- net M0_B: track 0.00 -> 69.4 mm
- net M0_A: track 0.00 -> 57.6 mm
- net PV+: track 0.00 -> 47.5 mm
- added copper zone on B.Cu, net GND
- added copper zone on F.Cu, net GND
Other:
- board size 144.3 x 127.8 mm -> 144.3 x 133.7 mm
- net class Default: trace_width 0.25 -> 0.381
- rule trace_min: 0.2 -> 0.127

Commit message: minor changes
Routing:
- net PV+: track 47.5 -> 48.9 mm
Changed lines of the file:
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@@
   )
   (setup
-    (last_trace_width 1.524)
+    (last_trace_width 2.54)
     (user_trace_width 0.508)
     (user_trace_width 0.762)
@@
   (segment (start 62.484 96.52) (end 40.64 74.676) (width 2.54) (layer B.Cu) (net 52))
   (segment (start 62.484 143.074) (end 62.484 96.52) (width 2.54) (layer B.Cu) (net 52))
-  (segment (start 43.179999 93.725999) (end 40.64 91.186) (width 2.54) (layer F.Cu) (net 60))
-  (segment (start 46.654001 97.200001) (end 43.179999 93.725999) (width 2.54) (layer F.Cu) (net 60))
-  (segment (start 46.654001 128.903999) (end 46.654001 97.200001) (width 2.54) (layer F.Cu) (net 60))
-  (segment (start 41.484 134.074) (end 46.654001 128.903999) (width 2.54) (layer F.Cu) (net 60))
+  (segment (start 43.179999 93.725999) (end 40.64 91.186) (width 2.54) (layer B.Cu) (net 60))
+  (segment (start 48.26 98.806) (end 43.179999 93.725999) (width 2.54) (layer B.Cu) (net 60))
+  (segment (start 48.26 127.298) (end 48.26 98.806) (width 2.54) (layer B.Cu) (net 60))
+  (segment (start 41.484 134.074) (end 48.26 127.298) (width 2.54) (layer B.Cu) (net 60))
   (zone (net 10) (net_name GND) (layer F.Cu) (hatch edge 0.508)
     (connect_pads (clearance 0.508))

Commit message: footprints made for resistor and odrive. Added IC to schematic
Parts:
- removed 50W2RJ1: 50W2RJ1, Footprints:PowerResistorMounts
- removed U1: ODrive, Footprints:ODriveInterfacingBoard
- added REF**: ODriveInterfacingBoard, Footprints:ODriveInterfacingBoard, F.Cu at (35.1, 174.2)
- moved D10 177.8 mm to (-13.4, 75.7)
- moved D12 177.8 mm to (-13.4, 78.7)
- moved D14 177.8 mm to (-13.4, 67.6)
- moved D15 177.8 mm to (-13.4, 70.6)
- moved D6 177.8 mm to (-13.4, 83.8)
- moved D8 177.8 mm to (-13.4, 86.9)
- moved R6 177.8 mm to (-22.7, 69.6)
- moved D13 163.2 mm to (213.0, 94.9)
- moved D11 163.2 mm to (212.8, 90.8)
- moved D3 163.2 mm to (210.8, 77.1)
- moved D5 163.2 mm to (210.8, 80.1)
- moved D7 163.2 mm to (210.4, 83.7)
- moved D9 163.2 mm to (211.3, 86.7)
- moved D1 153.3 mm to (227.1, 59.3)
- moved D2 153.3 mm to (267.7, 62.4)
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Connections:
- Conn14 pad 1: +3V3 -> Net-(Conn14-Pad1)
- Conn14 pad 2: +5V -> Net-(Conn14-Pad2)
- Conn14 pad 4: /Tx -> (no net)
- Conn14 pad 5: /Rx -> (no net)
- Conn2 pad 5: Net-(Conn2-Pad5) -> GND
- Conn3 pad 2: PV+ -> (no net)
Routing:
- net M1_A: track 101.1 -> 0.00 mm
- net M1_B: track 89.3 -> 0.00 mm
- net M0_C: track 81.2 -> 0.00 mm
- net Net-(50W2RJ1-Pad1): track 81.2 -> 0.00 mm
- net M1_C: track 77.4 -> 0.00 mm
- net Net-(50W2RJ1-Pad2): track 73.6 -> 0.00 mm
- net M0_B: track 69.4 -> 0.00 mm
- net M0_A: track 57.6 -> 0.00 mm
- net PV+: track 48.9 -> 0.00 mm
Other:
- outline, holes or cut-outs redrawn

Commit message: finished traces of everything except LEDs
Parts:
- removed Conn14: Molex_SL_05, MRDT_Connectors:MOLEX_SL_05_Horizontal
- removed REF**: ODriveInterfacingBoard, Footprints:ODriveInterfacingBoard
- added 50W2RJ1: 50W2RJ1, Footprints:PowerResistorMounts, F.Cu at (107.4, 81.3)
- added C1: .1u, Capacitor_SMD:C_0603_1608Metric_Pad1.05x0.95mm_HandSolder, F.Cu at (101.6, 63.8)
- added Conn10: Molex_SL_05, MRDT_Connectors:MOLEX_SL_05_Horizontal, F.Cu at (107.2, 53.8)
- added Conn9: Molex_SL_03, MRDT_Connectors:MOLEX_SL_03_Horizontal, F.Cu at (92.5, 53.8)
- added R16: 0, Resistor_SMD:R_0603_1608Metric_Pad1.05x0.95mm_HandSolder, F.Cu at (138.9, 140.6)
- added R17: 0, Resistor_SMD:R_0603_1608Metric_Pad1.05x0.95mm_HandSolder, F.Cu at (136.3, 140.6)
- added R18: 120, Resistor_SMD:R_0603_1608Metric_Pad1.05x0.95mm_HandSolder, F.Cu at (103.4, 56.1)
- added U1: ODrive, Footprints:ODriveInterfacingBoard, F.Cu at (35.1, 174.2)
- added U2: MAX3077E, Package_SO:SOIC-8_3.9x4.9mm_P1.27mm, F.Cu at (103.6, 59.9)
- Conn13: footprint MRDT_Connectors:MOLEX_SL_09_Horizontal -> MRDT_Connectors:MOLEX_SL_09_Vertical
- Conn2: footprint MRDT_Connectors:MOLEX_SL_05_Horizontal -> MRDT_Connectors:MOLEX_SL_05_Vertical
- Conn3: footprint MRDT_Connectors:Anderson_2_Horizontal_Side_by_Side -> MRDT_Connectors:Anderson_2_Horizontal_Stacked
- moved D11 188.6 mm to (78.2, -41.3)
- moved R1 188.6 mm to (116.1, -11.7)
- moved R13 188.6 mm to (123.3, -6.94)
- moved R5 188.6 mm to (96.8, -9.14)
- moved R7 188.6 mm to (93.2, -3.56)
- moved R9 188.6 mm to (109.7, -5.35)
- moved D13 188.6 mm to (78.4, -37.2)
- moved D3 188.6 mm to (76.2, -55.0)
- moved D5 188.6 mm to (76.2, -51.9)
- moved D7 188.6 mm to (75.8, -48.4)
- moved D9 188.6 mm to (76.7, -45.3)
- moved R10 188.6 mm to (118.2, -21.3)
- moved R11 188.6 mm to (127.9, -17.8)
- moved R12 188.6 mm to (120.0, -6.04)
- moved R14 188.6 mm to (126.7, -6.94)
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Connections:
- net /E0_3V3 renamed Net-(Conn5-Pad1)
- net /E1_3V3 renamed Net-(Conn4-Pad1)
- Conn13 pad 1: /GPIO_3 -> GPIO_8
- Conn13 pad 2: /GPIO_4 -> GPIO_7
- Conn13 pad 3: /GPIO_5 -> GPIO_6
- Conn13 pad 4: /GPIO_6 -> GPIO_5
- Conn13 pad 5: /GPIO_7 -> GPIO_4
- Conn13 pad 6: /GPIO_8 -> GPIO_3
- Conn2 pad 3: /CAN_H -> CAN_H
- Conn2 pad 4: /CAN_R -> CAN_L
- Conn3 pad 1: GND -> PV+
- Conn4 pad 2: /E1_5V -> GND
- Conn4 pad 3: /E1_A -> /E1_Z
- Conn4 pad 5: /E1_Z -> /E1_A
- Conn4 pad 6: /E1_GND -> +5V
- Conn4 pad 7: Net-(Conn4-Pad7) -> +3V3
- Conn5 pad 2: /E0_5V -> GND
- Conn5 pad 3: /E0_A -> /E0_Z
- Conn5 pad 5: /E0_Z -> /E0_A
- Conn5 pad 6: /E0_GND -> +5V
- Conn5 pad 7: Net-(Conn5-Pad7) -> +3V3
- Conn6 pad 4: /SCK -> MOSI
- Conn6 pad 5: /MISO -> MISO
- Conn6 pad 6: /MOSI -> SCK
- Conn7 pad 1: M0_A -> M0_C
- Conn7 pad 3: M0_C -> M0_A
- Conn8 pad 1: M1_A -> M1_C
- Conn8 pad 3: M1_C -> M1_A
Routing:
- net +3V3: track 0.00 -> 331.1 mm, vias 0 -> 6
- net +5V: track 0.00 -> 240.1 mm, vias 0 -> 3
- net Net-(Conn1-Pad2): track 0.00 -> 154.4 mm, vias 0 -> 3
- net Net-(Conn1-Pad1): track 0.00 -> 151.5 mm, vias 0 -> 3
- net Rx: track 0.00 -> 147.0 mm, vias 0 -> 4
- net Tx: track 0.00 -> 145.7 mm, vias 0 -> 4
- net SCK: track 0.00 -> 142.2 mm, vias 0 -> 3
- net MISO: track 0.00 -> 141.9 mm, vias 0 -> 3
- net MOSI: track 0.00 -> 140.4 mm, vias 0 -> 3
- net CAN_H: track 0.00 -> 139.4 mm, vias 0 -> 2
- net CAN_L: track 0.00 -> 135.3 mm, vias 0 -> 2
- net /E0_Z: track 0.00 -> 133.5 mm
- net /E0_B: track 0.00 -> 129.7 mm
- net /E0_A: track 0.00 -> 126.0 mm
- net GPIO_3: track 0.00 -> 124.3 mm
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Other:
- outline, holes or cut-outs redrawn

Commit message: via stitching added
Parts:
- moved D10 231.3 mm to (229.4, 123.4)
- moved D12 231.3 mm to (229.4, 126.5)
- moved D14 231.3 mm to (229.4, 115.3)
- moved D15 231.3 mm to (229.4, 118.4)
- moved D6 231.3 mm to (229.4, 131.6)
- moved D8 231.3 mm to (229.4, 134.6)
- moved R6 231.3 mm to (220.1, 117.3)
- moved D11 209.4 mm to (231.9, 101.0)
- moved D13 209.4 mm to (232.0, 105.0)
- moved D7 209.4 mm to (229.5, 93.9)
- moved D9 209.4 mm to (230.4, 96.9)
- moved D3 209.4 mm to (229.9, 87.2)
- moved D5 209.4 mm to (229.9, 90.3)
- moved R11 192.4 mm to (277.7, 102.9)
- moved R12 192.4 mm to (269.8, 114.6)
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Routing:
- net +3V3: track 331.1 -> 331.9 mm
- net +5V: track 240.1 -> 240.7 mm
- net GND: vias 34 -> 187

Commit message: Added LEDs for comm and Low Motor Phases
Parts:
- moved D4 235.0 mm to (53.3, 62.5), turned to 180 degrees
- moved D1 223.5 mm to (53.3, 68.1), turned to 180 degrees
- moved D2 218.8 mm to (53.3, 65.3), turned to 180 degrees
- moved R12 207.8 mm to (62.1, 107.3), turned to 180 degrees
- moved D8 203.4 mm to (37.7, 66.5)
- moved R15 203.4 mm to (71.5, 107.3), turned to 180 degrees
- moved D6 203.0 mm to (37.7, 64.5)
- moved R8 198.7 mm to (52.6, 107.3), turned to 180 degrees
- moved D12 196.2 mm to (42.5, 66.5)
- moved D10 195.9 mm to (42.5, 64.5)
- moved D15 188.7 mm to (47.9, 66.5)
- moved D14 188.5 mm to (47.9, 64.5)
- moved D5 171.7 mm to (59.8, 66.5)
- moved D3 171.6 mm to (59.8, 64.5)
- moved D9 168.2 mm to (64.9, 66.5)
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Connections:
- Conn10 pad 3: Net-(Conn10-Pad3) -> GND
- Conn10 pad 5: GND -> Net-(Conn10-Pad5)
- Conn4 pad 2: GND -> /E1_GND
- Conn5 pad 2: GND -> /E0_GND
- Conn9 pad 1: Rx -> Tx
- Conn9 pad 2: Tx -> GND
- Conn9 pad 3: GND -> Rx
- R1 pad 1: GPIO1 -> Tx
- R2 pad 1: GPIO2 -> Rx
- U2 pad 5: Net-(Conn10-Pad4) -> Net-(Conn10-Pad5)
- U2 pad 6: Net-(Conn10-Pad3) -> Net-(Conn10-Pad4)
Routing:
- net Net-(D13-Pad2): track 0.00 -> 165.8 mm, vias 0 -> 2
- net Net-(D9-Pad2): track 0.00 -> 156.3 mm, vias 0 -> 2
- net Net-(D5-Pad2): track 0.00 -> 144.3 mm, vias 0 -> 2
- net Net-(D4-Pad2): track 0.00 -> 121.0 mm, vias 0 -> 2
- net Net-(D2-Pad2): track 0.00 -> 120.9 mm, vias 0 -> 2
- net Net-(D1-Pad2): track 0.00 -> 118.9 mm, vias 0 -> 2
- net Net-(D15-Pad2): track 0.00 -> 75.3 mm, vias 0 -> 2
- net Net-(D12-Pad2): track 0.00 -> 63.9 mm, vias 0 -> 2
- net Net-(D8-Pad2): track 0.00 -> 60.3 mm, vias 0 -> 2
- net PV+: track 99.2 -> 120.6 mm
- net Net-(Conn10-Pad5): track 0.00 -> 13.3 mm
- net M0_C: track 72.8 -> 83.5 mm
- net Net-(Conn10-Pad3): track 9.77 -> 0.00 mm
- net +3V3: track 331.9 -> 340.8 mm
- net M1_A: track 85.0 -> 93.7 mm
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Other:
- board text added: "3V3"
- board text added: "A"
- board text added: "B"
- board text added: "C"
- board text added: "Comm"
- board text added: "M0(Left)"
- board text added: "M1(Right)"
- board text added: "Rx"
- board text added: "Tx"

Commit message: ADDED SILKSCREEN
Parts:
- added G***: LOGO, MRDT_Silkscreens:0_MRDT_Retro_Logo_34mmX21.5mm, F.Cu at (55.9, 160.0)
Routing:
- net GND: vias 149 -> 163
Other:
- board text added: "ODRIVE INTERFACING BOARD, REV. 1 MARS ROVER DESIGN TEAM MISSOURI S&T, 2019 BRIAN DAHLMAN"
