File: ODriveInterfacingBoard/ODriveInterfacingBoard.sch (KiCad schematic (older format))
At the start: 16 parts, among them U1 ODrive

Commit message: started the ODrive footprint
Parts:
- added D1: Tx Yellow, symbol Device:LED
- added D10: M0 B High Orange, symbol Device:LED
- added D11: M1 C High Orange, symbol Device:LED
- added D12: M0 B Low Orange, symbol Device:LED
- added D13: M1 C Low Orange, symbol Device:LED
- added D14: M0 C High Orange, symbol Device:LED
- added D15: M0 C Low Orange, symbol Device:LED
- added D2: Rx Yellow, symbol Device:LED
- added D3: M1 A High Orange, symbol Device:LED
- added D4: 3v3 Green, symbol Device:LED
- added D5: M1 A Low Orange, symbol Device:LED
- added D6: M0 A High Orange, symbol Device:LED
- added D7: M1 B High Orange, symbol Device:LED
- added D8: M0 A Low Orange, symbol Device:LED
- added D9: M1 B Low Orange, symbol Device:LED
- added R1, R10, R11, R12, R13, R14, R15, R2, R3, R4, R5, R6, R7, R8, R9: 1.5k, symbol Device:R
Connections:
- net labels added: GPIO1, GPIO2, M1_C
- wire segments 66 -> 111
Other:
- note added: "Indicators"

Commit message: footprint progress
Parts:
- removed U1: ODrive, symbol ODrive1x18Header:ODrive
- added U1: ODrive, symbol ODrive:ODrive
- 50W2RJ1: footprint (none) -> Footprints:PowerResistorMounts
- Conn1: footprint (none) -> MRDT_Connectors:MOLEX_SL_02_Horizontal
- Conn13: footprint (none) -> MRDT_Connectors:MOLEX_SL_09_Horizontal
- Conn14, Conn2: footprint (none) -> MRDT_Connectors:MOLEX_SL_05_Horizontal
- Conn3: footprint (none) -> MRDT_Connectors:Anderson_2_Vertical_Sidy_by_Side
- Conn4, Conn5, Conn6: footprint (none) -> MRDT_Connectors:MOLEX_SL_07_Horizontal
- Conn7: renamed from Conn8; value M0_B -> M0_A; footprint (none) -> MRDT_Connectors:Anderson_3_Vertical_Side_by_Side
- Conn7: renamed from Conn9; value M0_C -> M0_A; footprint (none) -> MRDT_Connectors:Anderson_3_Vertical_Side_by_Side
- Conn7: footprint (none) -> MRDT_Connectors:Anderson_3_Vertical_Side_by_Side
- Conn8: renamed from Conn11; value M1_B -> M1_A; footprint (none) -> MRDT_Connectors:Anderson_3_Vertical_Side_by_Side
- Conn8: renamed from Conn10; footprint (none) -> MRDT_Connectors:Anderson_3_Vertical_Side_by_Side
- Conn8: renamed from Conn12; value M1_C -> M1_A; footprint (none) -> MRDT_Connectors:Anderson_3_Vertical_Side_by_Side
- D1, D10, D11, D12, D13, D14, D15, D2, D3, D4, D5, D6, D7, D8, D9: footprint (none) -> LED_SMD:LED_0603_1608Metric_Pad1.05x0.95mm_HandSolder
- R1, R10, R11, R12, R13, R14, R15, R2, R3, R4, R5, R6, R7, R8, R9: footprint (none) -> Resistor_SMD:R_0603_1608Metric_Pad1.05x0.95mm_HandSolder

Commit message: finished footprints started layout
Parts:
- Conn3: footprint MRDT_Connectors:Anderson_2_Vertical_Sidy_by_Side -> MRDT_Connectors:Anderson_2_Horizontal_Side_by_Side
- Conn7, Conn8: footprint MRDT_Connectors:Anderson_3_Vertical_Side_by_Side -> MRDT_Connectors:Anderson_3_Horizontal_Side_by_Side
- U1: footprint (none) -> Footprints:ODriveInterfacingBoard
Changed lines of the file:
@@
 F 0 "Conn3" H 1650 3850 60  0000 C CNN
 F 1 "AndersonPP" H 1650 3950 60  0000 C CNN
-F 2 "MRDT_Connectors:Anderson_2_Vertical_Sidy_by_Side" H 1850 3250 60  0001 C CNN
+F 2 "MRDT_Connectors:Anderson_2_Horizontal_Side_by_Side" H 1850 3250 60  0001 C CNN
 F 3 "" H 1850 3250 60  0001 C CNN
 	1    2000 3800
@@
 F 0 "Conn7" H 3500 3500 60  0000 C CNN
 F 1 "M0_A" H 3673 3603 60  0000 R CNN
-F 2 "MRDT_Connectors:Anderson_3_Vertical_Side_by_Side" H 3550 2900 60  0001 C CNN
+F 2 "MRDT_Connectors:Anderson_3_Horizontal_Side_by_Side" H 3550 2900 60  0001 C CNN
 F 3 "" H 3550 2900 60  0001 C CNN
 	2    3700 3450
@@
 F 0 "Conn7" H 3350 3750 60  0000 L CNN
 F 1 "M0_A" H 3672 3853 60  0000 R CNN
-F 2 "MRDT_Connectors:Anderson_3_Vertical_Side_by_Side" H 3550 3150 60  0001 C CNN
+F 2 "MRDT_Connectors:Anderson_3_Horizontal_Side_by_Side" H 3550 3150 60  0001 C CNN
 F 3 "" H 3550 3150 60  0001 C CNN
 	3    3700 3700
@@
 F 0 "Conn7" H 3673 3247 60  0000 R CNN
 F 1 "M0_A" H 3673 3353 60  0000 R CNN
-F 2 "MRDT_Connectors:Anderson_3_Vertical_Side_by_Side" H 3550 2650 60  0001 C CNN
+F 2 "MRDT_Connectors:Anderson_3_Horizontal_Side_by_Side" H 3550 2650 60  0001 C CNN
 F 3 "" H 3550 2650 60  0001 C CNN
 	1    3700 3200
@@
 F 0 "Conn8" H 3500 4250 60  0000 C CNN
 F 1 "M1_A" H 3672 4353 60  0000 R CNN
-F 2 "MRDT_Connectors:Anderson_3_Vertical_Side_by_Side" H 3550 3650 60  0001 C CNN
+F 2 "MRDT_Connectors:Anderson_3_Horizontal_Side_by_Side" H 3550 3650 60  0001 C CNN
 F 3 "" H 3550 3650 60  0001 C CNN
 	2    3700 4200
@@
 F 0 "Conn8" H 3672 3997 60  0000 R CNN
 F 1 "M1_A" H 3672 4103 60  0000 R CNN
-F 2 "MRDT_Connectors:Anderson_3_Vertical_Side_by_Side" H 3550 3400 60  0001 C CNN
+F 2 "MRDT_Connectors:Anderson_3_Horizontal_Side_by_Side" H 3550 3400 60  0001 C CNN
 F 3 "" H 3550 3400 60  0001 C CNN
 	1    3700 3950
@@
 F 0 "Conn8" H 3300 4500 60  0000 L CNN
 F 1 "M1_A" H 3672 4603 60  0000 R CNN
-F 2 "MRDT_Connectors:Anderson_3_Vertical_Side_by_Side" H 3550 3900 60  0001 C CNN
+F 2 "MRDT_Connectors:Anderson_3_Horizontal_Side_by_Side" H 3550 3900 60  0001 C CNN
 F 3 "" H 3550 3900 60  0001 C CNN
 	3    3700 4450
@@
 F 0 "Conn3" H 2206 3937 60  0000 C CNN
 F 1 "AndersonPP" H 2206 3831 60  0000 C CNN
-F 2 "MRDT_Connectors:Anderson_2_Vertical_Sidy_by_Side" H 1850 3000 60  0001 C CNN
+F 2 "MRDT_Connectors:Anderson_2_Horizontal_Side_by_Side" H 1850 3000 60  0001 C CNN
 F 3 "" H 1850 3000 60  0001 C CNN
 	4    2000 3550
@@
 M1_B
 Text Label 3100 4550 0    49   ~ 0
-M1_B
+M1_C
 Wire Notes Line
 	10250 450  10300 450
@@
 F 0 "U1" H 2850 5515 50  0000 C CNN
 F 1 "ODrive" H 2850 5424 50  0000 C CNN
-F 2 "" H 3150 3450 50  0001 C CNN
+F 2 "Footprints:ODriveInterfacingBoard" H 3150 3450 50  0001 C CNN
 F 3 "" H 3150 3450 50  0001 C CNN
 	2    2700 3250
@@
 F 0 "U1" H 2850 6115 50  0000 C CNN
 F 1 "ODrive" H 2850 6024 50  0000 C CNN
-F 2 "" H 3300 4800 50  0001 C CNN
+F 2 "Footprints:ODriveInterfacingBoard" H 3300 4800 50  0001 C CNN
 F 3 "" H 3300 4800 50  0001 C CNN
 	1    2850 4600

Commit message: footprints made for resistor and odrive. Added IC to schematic
Parts:
- added C1: 10u, Capacitor_SMD:C_0603_1608Metric_Pad1.05x0.95mm_HandSolder, symbol Device:C
- added Conn9: Molex_SL_04, MRDT_Connectors:MOLEX_SL_04_Horizontal, symbol MRDT_Connectors:Molex_SL_04
- added R16, R17: 0, Resistor_SMD:R_0603_1608Metric_Pad1.05x0.95mm_HandSolder, symbol Device:R
- added U2: MAX3077E, Package_SO:SOIC-8_3.9x4.9mm_P1.27mm, symbol MRDT_ICs:MAX3077E
- Conn14: symbol MRDT_Connectors:Molex_SL_05 -> MRDT_Connectors:Molex_SL_03
Connections:
- net labels added: CAN_L, power:+3V3, power:GND
- net labels removed: CAN_R
- wire segments 111 -> 132
- no-connect marks 4 -> 3
Other:
- moved on the sheet: 50W2RJ1, Conn1, Conn13, Conn2, Conn3A, Conn3D, Conn4, Conn5, Conn6, Conn7A, Conn7B, Conn7C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

Commit message: finished traces of everything except LEDs
Parts:
- removed Conn14: Molex_SL_05, MRDT_Connectors:MOLEX_SL_05_Horizontal, symbol MRDT_Connectors:Molex_SL_03
- removed Conn9: Molex_SL_04, MRDT_Connectors:MOLEX_SL_04_Horizontal, symbol MRDT_Connectors:Molex_SL_04
- added Conn10: Molex_SL_05, MRDT_Connectors:MOLEX_SL_05_Horizontal, symbol MRDT_Connectors:Molex_SL_05
- added Conn9: Molex_SL_03, MRDT_Connectors:MOLEX_SL_03_Horizontal, symbol MRDT_Connectors:Molex_SL_03
- added R18: 120, Resistor_SMD:R_0603_1608Metric_Pad1.05x0.95mm_HandSolder, symbol Device:R
- C1: value 10u -> .1u
- Conn13: footprint MRDT_Connectors:MOLEX_SL_09_Horizontal -> MRDT_Connectors:MOLEX_SL_09_Vertical
- Conn2: footprint MRDT_Connectors:MOLEX_SL_05_Horizontal -> MRDT_Connectors:MOLEX_SL_05_Vertical
- Conn3: footprint MRDT_Connectors:Anderson_2_Horizontal_Side_by_Side -> MRDT_Connectors:Anderson_2_Horizontal_Stacked
Connections:
- wire segments 132 -> 148
Changed lines of the file:
@@
 $Comp
 L MRDT_Connectors:AndersonPP Conn3
-U 1 1 5C728113
+U 4 1 5C728113
 P 2050 6650
 F 0 "Conn3" H 1700 6700 60  0000 C CNN
 F 1 "AndersonPP" H 1700 6800 60  0000 C CNN
-F 2 "MRDT_Connectors:Anderson_2_Horizontal_Side_by_Side" H 1900 6100 60  0001 C CNN
+F 2 "MRDT_Connectors:Anderson_2_Horizontal_Stacked" H 1900 6100 60  0001 C CNN
 F 3 "" H 1900 6100 60  0001 C CNN
-	1    2050 6650
+	4    2050 6650
 	1    0    0    -1
 $EndComp
@@
 $Comp
 L MRDT_Connectors:AndersonPP Conn7
-U 3 1 5C7282A5
+U 1 1 5C7282A5
 P 3750 6550
 F 0 "Conn7" H 3400 6600 60  0000 L CNN
@@
 F 2 "MRDT_Connectors:Anderson_3_Horizontal_Side_by_Side" H 3600 6000 60  0001 C CNN
 F 3 "" H 3600 6000 60  0001 C CNN
-	3    3750 6550
+	1    3750 6550
 	-1   0    0    1
 $EndComp
 $Comp
 L MRDT_Connectors:AndersonPP Conn7
-U 1 1 5C7282C7
+U 3 1 5C7282C7
 P 3750 6050
 F 0 "Conn7" H 3723 6097 60  0000 R CNN
@@
 F 2 "MRDT_Connectors:Anderson_3_Horizontal_Side_by_Side" H 3600 5500 60  0001 C CNN
 F 3 "" H 3600 5500 60  0001 C CNN
-	1    3750 6050
+	3    3750 6050
 	-1   0    0    1
 $EndComp
@@
 $Comp
 L MRDT_Connectors:AndersonPP Conn8
-U 1 1 5C728323
+U 3 1 5C728323
 P 3750 6800
 F 0 "Conn8" H 3722 6847 60  0000 R CNN
@@
 F 2 "MRDT_Connectors:Anderson_3_Horizontal_Side_by_Side" H 3600 6250 60  0001 C CNN
 F 3 "" H 3600 6250 60  0001 C CNN
-	1    3750 6800
+	3    3750 6800
 	-1   0    0    1
 $EndComp
 $Comp
 L MRDT_Connectors:AndersonPP Conn8
-U 3 1 5C728351
+U 1 1 5C728351
 P 3750 7300
 F 0 "Conn8" H 3350 7350 60  0000 L CNN
@@
 F 2 "MRDT_Connectors:Anderson_3_Horizontal_Side_by_Side" H 3600 6750 60  0001 C CNN
 F 3 "" H 3600 6750 60  0001 C CNN
-	3    3750 7300
+	1    3750 7300
 	-1   0    0    1
 $EndComp
@@
 $Comp
 L MRDT_Connectors:AndersonPP Conn3
-U 4 1 5C72CC94
+U 1 1 5C72CC94
 P 2050 6400
 F 0 "Conn3" H 2256 6787 60  0000 C CNN
 F 1 "AndersonPP" H 2256 6681 60  0000 C CNN
-F 2 "MRDT_Connectors:Anderson_2_Horizontal_Side_by_Side" H 1900 5850 60  0001 C CNN
+F 2 "MRDT_Connectors:Anderson_2_Horizontal_Stacked" H 1900 5850 60  0001 C CNN
 F 3 "" H 1900 5850 60  0001 C CNN
-	4    2050 6400
+	1    2050 6400
 	1    0    0    -1
 $EndComp
@@
 L MRDT_Connectors:Molex_SL_07 Conn4
 U 1 1 5C72DB74
-P 1800 3350
-F 0 "Conn4" H 1744 4247 60  0000 C CNN
-F 1 "Molex_SL_07" H 1744 4141 60  0000 C CNN
-F 2 "MRDT_Connectors:MOLEX_SL_07_Horizontal" H 1800 3550 60  0001 C CNN
-F 3 "" H 1800 3550 60  0001 C CNN
-	1    1800 3350
-	-1   0    0    -1
+P 1800 2650
+F 0 "Conn4" H 1744 3547 60  0000 C CNN
+F 1 "Molex_SL_07" H 1744 3441 60  0000 C CNN
+F 2 "MRDT_Connectors:MOLEX_SL_07_Horizontal" H 1800 2850 60  0001 C CNN
+F 3 "" H 1800 2850 60  0001 C CNN
+	1    1800 2650
+	-1   0    0    1
 $EndComp
 $Comp
 L MRDT_Connectors:Molex_SL_07 Conn5
 U 1 1 5C72DD01
-P 3000 3350
-F 0 "Conn5" H 3150 3400 60  0000 L CNN
-F 1 "Molex_SL_07" V 3050 3400 60  0000 L CNN
-F 2 "MRDT_Connectors:MOLEX_SL_07_Horizontal" H 3000 3550 60  0001 C CNN
-F 3 "" H 3000 3550 60  0001 C CNN
-	1    3000 3350
-	1    0    0    -1
+P 3000 2650
+F 0 "Conn5" H 3150 2700 60  0000 L CNN
+F 1 "Molex_SL_07" V 3050 2700 60  0000 L CNN
+F 2 "MRDT_Connectors:MOLEX_SL_07_Horizontal" H 3000 2850 60  0001 C CNN
+F 3 "" H 3000 2850 60  0001 C CNN
+	1    3000 2650
+	1    0    0    1
 $EndComp
 Wire Wire Line
@@
 U 1 1 5C732A4C
 P 4750 3000
-F 0 "Conn6" V 4877 3408 60  0000 L CNN
+F 0 "Conn6" V 5050 3400 60  0000 L CNN
 F 1 "Molex_SL_07" V 4877 3302 60  0000 L CNN
 F 2 "MRDT_Connectors:MOLEX_SL_07_Horizontal" H 4750 3200 60  0001 C CNN
@@
 F 0 "Conn2" H 644 3197 60  0000 C CNN
 F 1 "Molex_SL_05" H 644 3091 60  0000 C CNN
-F 2 "MRDT_Connectors:MOLEX_SL_05_Horizontal" H 700 2500 60  0001 C CNN
+F 2 "MRDT_Connectors:MOLEX_SL_05_Vertical" H 700 2500 60  0001 C CNN
 F 3 "" H 700 2500 60  0001 C CNN
 	1    700  2500
@@
 	2100 2050 2100 2000
 $Comp
-L MRDT_Connectors:Molex_SL_03 Conn14
-U 1 1 5C7435B7
-P 4750 1750
-F 0 "Conn14" H 4877 2058 60  0000 L CNN
-F 1 "Molex_SL_05" H 4877 1952 60  0000 L CNN
-F 2 "MRDT_Connectors:MOLEX_SL_05_Horizontal" H 4750 1750 60  0001 C CNN
-F 3 "" H 4750 1750 60  0001 C CNN
-	1    4750 1750
-	1    0    0    -1
-$EndComp
-$Comp
 L power:GND #PWR013
 U 1 1 5C74723B
-P 4500 1700
-F 0 "#PWR013" H 4500 1450 50  0001 C CNN
-F 1 "GND" V 4505 1572 50  0000 R CNN
-F 2 "" H 4500 1700 50  0001 C CNN
-F 3 "" H 4500 1700 50  0001 C CNN
-	1    4500 1700
-	1    0    0    -1
-$EndComp
-Wire Wire Line
-	4550 1700 4500 1700
+P 4500 1900
+F 0 "#PWR013" H 4500 1650 50  0001 C CNN
+F 1 "GND" V 4505 1772 50  0000 R CNN
+F 2 "" H 4500 1900 50  0001 C CNN
+F 3 "" H 4500 1900 50  0001 C CNN
+	1    4500 1900
+	1    0    0    -1
+$EndComp
+Wire Wire Line
+	4550 1900 4500 1900
 $Comp
 L power:+3V3 #PWR04
@@
 F 0 "Conn13" H 4877 4558 60  0000 L CNN
 F 1 "Molex_SL_09" H 4877 4452 60  0000 L CNN
-F 2 "MRDT_Connectors:MOLEX_SL_09_Horizontal" H 4750 4450 60  0001 C CNN
+F 2 "MRDT_Connectors:MOLEX_SL_09_Vertical" H 4750 4450 60  0001 C CNN
 F 3 "" H 4750 4450 60  0001 C CNN
 	1    4750 4050
@@
 L MRDT_Connectors:Molex_SL_02 Conn1
 U 1 1 5C75A9EC
-P 1750 1850
-F 0 "Conn1" H 1850 2250 60  0000 C CNN
-F 1 "Molex_SL_02" H 1850 2150 60  0000 C CNN
-F 2 "MRDT_Connectors:MOLEX_SL_02_Horizontal" H 1750 1750 60  0001 C CNN
-F 3 "" H 1750 1750 60  0001 C CNN
-	1    1750 1850
-	-1   0    0    -1
+P 1750 1650
+F 0 "Conn1" H 1850 2050 60  0000 C CNN
+F 1 "Molex_SL_02" H 1850 1950 60  0000 C CNN
+F 2 "MRDT_Connectors:MOLEX_SL_02_Horizontal" H 1750 1550 60  0001 C CNN
+F 3 "" H 1750 1550 60  0001 C CNN
+	1    1750 1650
+	-1   0    0    1
 $EndComp
 Wire Wire Line
@@
 P 3550 1000
 F 0 "C1" H 3350 1050 50  0000 L CNN
-F 1 "10u" H 3300 950 50  0000 L CNN
+F 1 ".1u" H 3300 950 50  0000 L CNN
 F 2 "Capacitor_SMD:C_0603_1608Metric_Pad1.05x0.95mm_HandSolder" H 3588 850 50  0001 C CNN
 F 3 "~" H 3550 1000 50  0001 C CNN
@@
 Wire Wire Line
 	3900 850  3900 800
-$Comp
-L MRDT_Connectors:Molex_SL_04 Conn9
-U 1 1 5C818822
-P 4750 1200
-F 0 "Conn9" H 4877 1458 60  0000 L CNN
-F 1 "Molex_SL_04" H 4877 1352 60  0000 L CNN
-F 2 "MRDT_Connectors:MOLEX_SL_04_Horizontal" H 4750 1200 60  0001 C CNN
-F 3 "" H 4750 1200 60  0001 C CNN
-	1    4750 1200
-	1    0    0    -1
-$EndComp
 Text GLabel 3450 1800 2    50   Output ~ 0
 Tx
@@
 Rx
 Wire Wire Line
-	4450 850  4550 850
-Wire Wire Line
-	4550 950  4450 950
-Wire Wire Line
-	4450 1050 4550 1050
-Wire Wire Line
-	4550 1150 4450 1150
-Wire Wire Line
 	2650 1800 3050 1800
 Wire Wire Line
@@
 Wire Wire Line
 	3950 1050 3900 1050
-Text GLabel 4500 1500 0    50   Input ~ 0
+Text GLabel 4500 1800 0    50   Input ~ 0
 Tx
-Text GLabel 4500 1600 0    50   Output ~ 0
+Text GLabel 4500 1700 0    50   Output ~ 0
 Rx
 Wire Wire Line
-	4500 1500 4550 1500
-Wire Wire Line
-	4550 1600 4500 1600
+	4500 1700 4550 1700
+Wire Wire Line
+	4550 1800 4500 1800
 Text GLabel 2700 1500 2    50   Output ~ 0
 SCK
@@
 Wire Wire Line
 	2650 1700 2700 1700
-Text GLabel 4500 2650 0    50   Input ~ 0
+Text GLabel 4500 2850 0    50   Input ~ 0
 SCK
 Text GLabel 4500 2750 0    50   Input ~ 0
 MISO
-Text GLabel 4500 2850 0    50   Input ~ 0
+Text GLabel 4500 2650 0    50   Input ~ 0
 MOSI
 Wire Wire Line
@@
 Wire Wire Line
 	2750 2500 2650 2500
+Text GLabel 4450 3700 0    50   Input ~ 0
+GPIO_3
+Text GLabel 4450 3600 0    50   Input ~ 0
+GPIO_4
+Text GLabel 4450 3500 0    50   Input ~ 0
+GPIO_5
+Text GLabel 4450 3400 0    50   Input ~ 0
+GPIO_6
+Text GLabel 4450 3300 0    50   Input ~ 0
+GPIO_7
 Text GLabel 4450 3200 0    50   Input ~ 0
-GPIO_3
-Text GLabel 4450 3300 0    50   Input ~ 0
-GPIO_4
-Text GLabel 4450 3400 0    50   Input ~ 0
-GPIO_5
-Text GLabel 4450 3500 0    50   Input ~ 0
-GPIO_6
-Text GLabel 4450 3600 0    50   Input ~ 0
-GPIO_7
-Text GLabel 4450 3700 0    50   Input ~ 0
 GPIO_8
 Wire Wire Line
@@
 Wire Wire Line
 	2150 1800 1950 1800
+$Comp
+L ODriveInterfacingBoard-cache:power:GND #PWR0104
+U 1 1 5C98C91D
+P 5050 1300
+F 0 "#PWR0104" H 5050 1050 50  0001 C CNN
+F 1 "power:GND" H 5055 1127 50  0000 C CNN
+F 2 "" H 5050 1300 50  0001 C CNN
+F 3 "" H 5050 1300 50  0001 C CNN
+	1    5050 1300
+	1    0    0    -1
+$EndComp
+$Comp
+L Device:R R18
+U 1 1 5C98CA28
+P 4800 900
+F 0 "R18" H 4870 946 50  0000 L CNN
+F 1 "120" V 4800 850 50  0000 L CNN
+F 2 "Resistor_SMD:R_0603_1608Metric_Pad1.05x0.95mm_HandSolder" V 4730 900 50  0001 C CNN
+F 3 "~" H 4800 900 50  0001 C CNN
+	1    4800 900
+	-1   0    0    1
+$EndComp
+Wire Wire Line
+	4450 950  4700 950
+Wire Wire Line
+	4700 950  4700 1050
+Wire Wire Line
+	4700 1050 4800 1050
+Wire Wire Line
+	4700 850  4700 750
+Wire Wire Line
+	4700 750  4800 750
+Wire Wire Line
+	4450 850  4700 850
+Wire Wire Line
+	4800 750  4900 750
+Wire Wire Line
+	4900 750  4900 850
+Wire Wire Line
+	4900 850  5150 850
+Connection ~ 4800 750
+Wire Wire Line
+	4800 1050 4900 1050
+Wire Wire Line
+	4900 1050 4900 950
+Wire Wire Line
+	4900 950  5150 950
+Connection ~ 4800 1050
+Wire Wire Line
+	4650 1050 4650 1100
+Wire Wire Line
+	4650 1100 4950 1100
+Wire Wire Line
+	4950 1100 4950 1050
+Wire Wire Line
+	4950 1050 5150 1050
+Wire Wire Line
+	4450 1050 4650 1050
+Wire Wire Line
+	4450 1150 5150 1150
+Wire Wire Line
+	5150 1250 5050 1250
+Wire Wire Line
+	5050 1250 5050 1300
+$Comp
+L MRDT_Connectors:Molex_SL_03 Conn9
+U 1 1 5C9F2E94
+P 4750 1950
+F 0 "Conn9" H 4877 2158 60  0000 L CNN
+F 1 "Molex_SL_03" H 4877 2052 60  0000 L CNN
+F 2 "MRDT_Connectors:MOLEX_SL_03_Horizontal" H 4750 1950 60  0001 C CNN
+F 3 "" H 4750 1950 60  0001 C CNN
+	1    4750 1950
+	1    0    0    -1
+$EndComp
+$Comp
+L MRDT_Connectors:Molex_SL_05 Conn10
+U 1 1 5C9F30EB
+P 5350 1300
+F 0 "Conn10" H 5477 1608 60  0000 L CNN
+F 1 "Molex_SL_05" H 5477 1502 60  0000 L CNN
+F 2 "MRDT_Connectors:MOLEX_SL_05_Horizontal" H 5350 1300 60  0001 C CNN
+F 3 "" H 5350 1300 60  0001 C CNN
+	1    5350 1300
+	1    0    0    -1
+$EndComp
 $EndSCHEMATC

Commit message: Added LEDs for comm and Low Motor Phases
Connections:
- wire segments 148 -> 147
Changed lines of the file:
@@
 L power:GND #PWR013
 U 1 1 5C74723B
-P 4500 1900
-F 0 "#PWR013" H 4500 1650 50  0001 C CNN
-F 1 "GND" V 4505 1772 50  0000 R CNN
-F 2 "" H 4500 1900 50  0001 C CNN
-F 3 "" H 4500 1900 50  0001 C CNN
-	1    4500 1900
+P 4300 1800
+F 0 "#PWR013" H 4300 1550 50  0001 C CNN
+F 1 "GND" V 4305 1672 50  0000 R CNN
+F 2 "" H 4300 1800 50  0001 C CNN
+F 3 "" H 4300 1800 50  0001 C CNN
+	1    4300 1800
 	1    0    0    -1
 $EndComp
@@
 	1    0    0    -1
 $EndComp
-$Comp
-L ODriveInterfacingBoard-cache:power:GND #PWR0101
-U 1 1 5C7B5819
-P 950 2500
-F 0 "#PWR0101" H 950 2250 50  0001 C CNN
-F 1 "power:GND" H 955 2327 50  0000 C CNN
-F 2 "" H 950 2500 50  0001 C CNN
-F 3 "" H 950 2500 50  0001 C CNN
-	1    950  2500
-	1    0    0    -1
-$EndComp
 Wire Wire Line
 	900  2450 950  2450
@@
 	1    0    0    -1
 $EndComp
-$Comp
-L ODriveInterfacingBoard-cache:power:GND #PWR0102
-U 1 1 5C804CD3
-P 3900 1200
-F 0 "#PWR0102" H 3900 950 50  0001 C CNN
-F 1 "power:GND" H 3905 1027 50  0000 C CNN
-F 2 "" H 3900 1200 50  0001 C CNN
-F 3 "" H 3900 1200 50  0001 C CNN
-	1    3900 1200
-	1    0    0    -1
-$EndComp
 Wire Wire Line
 	3950 1150 3900 1150
@@
 Wire Wire Line
 	3550 850  3900 850
-$Comp
-L ODriveInterfacingBoard-cache:power:+3V3 #PWR0103
-U 1 1 5C813C5F
-P 3900 800
-F 0 "#PWR0103" H 3900 650 50  0001 C CNN
-F 1 "power:+3V3" H 3915 973 50  0000 C CNN
-F 2 "" H 3900 800 50  0001 C CNN
-F 3 "" H 3900 800 50  0001 C CNN
-	1    3900 800
-	1    0    0    -1
-$EndComp
 Connection ~ 3900 850
 Wire Wire Line
@@
 Wire Wire Line
 	3950 1050 3900 1050
-Text GLabel 4500 1800 0    50   Input ~ 0
+Text GLabel 4500 1700 0    50   Input ~ 0
 Tx
-Text GLabel 4500 1700 0    50   Output ~ 0
+Text GLabel 4500 1900 0    50   Output ~ 0
 Rx
 Wire Wire Line
 	4500 1700 4550 1700
-Wire Wire Line
-	4550 1800 4500 1800
 Text GLabel 2700 1500 2    50   Output ~ 0
 SCK
@@
 	2150 1800 1950 1800
 $Comp
-L ODriveInterfacingBoard-cache:power:GND #PWR0104
-U 1 1 5C98C91D
-P 5050 1300
-F 0 "#PWR0104" H 5050 1050 50  0001 C CNN
-F 1 "power:GND" H 5055 1127 50  0000 C CNN
-F 2 "" H 5050 1300 50  0001 C CNN
-F 3 "" H 5050 1300 50  0001 C CNN
-	1    5050 1300
-	1    0    0    -1
-$EndComp
-$Comp
 L Device:R R18
 U 1 1 5C98CA28
@@
 Connection ~ 4800 1050
 Wire Wire Line
-	4650 1050 4650 1100
-Wire Wire Line
-	4650 1100 4950 1100
-Wire Wire Line
-	4950 1100 4950 1050
-Wire Wire Line
-	4950 1050 5150 1050
-Wire Wire Line
 	4450 1050 4650 1050
-Wire Wire Line
-	4450 1150 5150 1150
-Wire Wire Line
-	5150 1250 5050 1250
-Wire Wire Line
-	5050 1250 5050 1300
 $Comp
 L MRDT_Connectors:Molex_SL_03 Conn9
@@
 	1    0    0    -1
 $EndComp
+Wire Wire Line
+	4300 1800 4550 1800
+$Comp
+L ODriveInterfacingBoard-cache:power:GND #PWR0101
+U 1 1 5CA0D82E
+P 5100 1050
+F 0 "#PWR0101" H 5100 800 50  0001 C CNN
+F 1 "power:GND" V 5105 923 50  0000 R CNN
+F 2 "" H 5100 1050 50  0001 C CNN
+F 3 "" H 5100 1050 50  0001 C CNN
+	1    5100 1050
+	0    1    1    0
+$EndComp
+$Comp
+L ODriveInterfacingBoard-cache:power:+3V3 #PWR0102
+U 1 1 5CA0DA4A
+P 3900 800
+F 0 "#PWR0102" H 3900 650 50  0001 C CNN
+F 1 "power:+3V3" H 3915 973 50  0000 C CNN
+F 2 "" H 3900 800 50  0001 C CNN
+F 3 "" H 3900 800 50  0001 C CNN
+	1    3900 800
+	1    0    0    -1
+$EndComp
+$Comp
+L ODriveInterfacingBoard-cache:power:GND #PWR0103
+U 1 1 5CA0DB15
+P 3900 1200
+F 0 "#PWR0103" H 3900 950 50  0001 C CNN
+F 1 "power:GND" H 3905 1027 50  0000 C CNN
+F 2 "" H 3900 1200 50  0001 C CNN
+F 3 "" H 3900 1200 50  0001 C CNN
+	1    3900 1200
+	1    0    0    -1
+$EndComp
+Wire Wire Line
+	5100 1050 5150 1050
+Wire Wire Line
+	5150 1150 4650 1150
+Wire Wire Line
+	4650 1050 4650 1150
+Wire Wire Line
+	4450 1150 4550 1150
+Wire Wire Line
+	4550 1150 4550 1250
+Wire Wire Line
+	4550 1250 5150 1250
+$Comp
+L ODriveInterfacingBoard-cache:power:GND #PWR0104
+U 1 1 5CA296E8
+P 950 2500
+F 0 "#PWR0104" H 950 2250 50  0001 C CNN
+F 1 "power:GND" H 955 2327 50  0000 C CNN
+F 2 "" H 950 2500 50  0001 C CNN
+F 3 "" H 950 2500 50  0001 C CNN
+	1    950  2500
+	1    0    0    -1
+$EndComp
