File: ODriveInterfacingBoard/ODriveInterfacingBoard.sch (KiCad schematic (older format))
At the start: 30 parts, among them U1 ODrive

Commit message: r
Parts:
- Conn7: value ML_B -> ML
- Conn7: value ML_A -> ML
- Conn7: value ML_C -> ML
- Conn8: value MR_B -> MR
- Conn8: value MR_C -> MR
- Conn8: value MR_A -> MR
Changed lines of the file:
@@
 P 4550 1600
 F 0 "Conn7" H 4350 1650 60  0000 C CNN
-F 1 "ML_B" H 4523 1753 60  0000 R CNN
+F 1 "ML" H 4523 1753 60  0000 R CNN
 F 2 "MRDT_Connectors:Anderson_3_Horizontal_Side_by_Side" H 4400 1050 60  0001 C CNN
 F 3 "" H 4400 1050 60  0001 C CNN
@@
 P 4550 1850
 F 0 "Conn7" H 4523 1897 60  0000 R CNN
-F 1 "ML_C" H 4523 2003 60  0000 R CNN
+F 1 "ML" H 4523 2003 60  0000 R CNN
 F 2 "MRDT_Connectors:Anderson_3_Horizontal_Side_by_Side" H 4400 1300 60  0001 C CNN
 F 3 "" H 4400 1300 60  0001 C CNN
@@
 P 4550 2350
 F 0 "Conn8" H 4350 2400 60  0000 C CNN
-F 1 "MR_B" H 4522 2503 60  0000 R CNN
+F 1 "MR" H 4522 2503 60  0000 R CNN
 F 2 "MRDT_Connectors:Anderson_3_Horizontal_Side_by_Side" H 4400 1800 60  0001 C CNN
 F 3 "" H 4400 1800 60  0001 C CNN
@@
 P 4550 2600
 F 0 "Conn8" H 4522 2647 60  0000 R CNN
-F 1 "MR_C" H 4522 2753 60  0000 R CNN
+F 1 "MR" H 4522 2753 60  0000 R CNN
 F 2 "MRDT_Connectors:Anderson_3_Horizontal_Side_by_Side" H 4400 2050 60  0001 C CNN
 F 3 "" H 4400 2050 60  0001 C CNN
@@
 P 4550 2100
 F 0 "Conn8" H 4150 2150 60  0000 L CNN
-F 1 "MR_A" H 4522 2253 60  0000 R CNN
+F 1 "MR" H 4522 2253 60  0000 R CNN
 F 2 "MRDT_Connectors:Anderson_3_Horizontal_Side_by_Side" H 4400 1550 60  0001 C CNN
 F 3 "" H 4400 1550 60  0001 C CNN
@@
 P 4550 1350
 F 0 "Conn7" H 4200 1400 60  0000 L CNN
-F 1 "ML_A" H 4522 1503 60  0000 R CNN
+F 1 "ML" H 4522 1503 60  0000 R CNN
 F 2 "MRDT_Connectors:Anderson_3_Horizontal_Side_by_Side" H 4400 800 60  0001 C CNN
 F 3 "" H 4400 800 60  0001 C CNN

Commit message: Just need silks and vias, babam
Parts:
- added D16, D17, D18, D19, D20, D4: Rx Yellow, LED_SMD:LED_0603_1608Metric_Pad1.05x0.95mm_HandSolder, symbol ODriveInterfacingBoard-rescue:LED-Device
- added R11, R12, R13, R14, R4, R5: 500, Resistor_SMD:R_0603_1608Metric_Pad1.05x0.95mm_HandSolder, symbol ODriveInterfacingBoard-rescue:R-Device
Connections:
- net GND: now also Conn1.1, Conn2.1, U1.E0_GND, U1.E1_GND, D16.1 (K), D17.1 (K), D18.1 (K), D19.1 (K), D20.1 (K), D4.1 (K)
- net L_Encoder_5V: now also Conn1.4; no longer Conn1.1
- net L_Encoder_A: now also Conn1.3, R12.1; no longer Conn1.2
- net L_Encoder_B: now also Conn1.5, R13.1; no longer Conn1.3
- net L_Encoder_Z: now also Conn1.2, R14.1; no longer Conn1.4
- net R_Encoder_5V: now also Conn2.4; no longer Conn2.1
- net R_Encoder_A: now also Conn2.3, R4.1; no longer Conn2.2
- net R_Encoder_B: now also Conn2.5, R5.1; no longer Conn2.3
- net R_Encoder_Z: now also Conn2.2, R11.1; no longer Conn2.4
- removed net L_Encoder_Gnd: Conn1.5, U1.E0_GND
- removed net R_Encoder_Gnd: Conn2.5, U1.E1_GND
- new net: D4.2 (A), R4.2
- new net: D16.2 (A), R5.2
- new net: D17.2 (A), R11.2
- new net: D18.2 (A), R12.2
- new net: D19.2 (A), R13.2
- new net: D20.2 (A), R14.2
Other:
- moved on the sheet: D1, D10, D11, D12, D13, D14, D15, D2, D3, D5, D6, D7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

Commit message: https://www.youtube.com/watch?v=dQw4w9WgXcQ
Parts:
- 50W2RJ1, R1, R10, R11, R12, R13, R14, R2, R3, R4, R5, R6, R7, R8, R9: symbol ODriveInterfacingBoard-rescue:R-Device -> ODriveInterfacingBoard-rescue:R-Device-ODriveInterfacingBoard-rescue
- Conn3, Conn7, Conn8: symbol ODriveInterfacingBoard-rescue:AndersonPP-MRDT_Connectors -> ODriveInterfacingBoard-rescue:AndersonPP-MRDT_Connectors-ODriveInterfacingBoard-rescue
- Conn9: symbol ODriveInterfacingBoard-rescue:Molex_SL_03-MRDT_Connectors -> ODriveInterfacingBoard-rescue:Molex_SL_03-MRDT_Connectors-ODriveInterfacingBoard-rescue
- D1, D10, D11, D12, D13, D14, D15, D16, D17, D18, D19, D2, D20, D3, D4, D5, D6, D7, D8, D9: symbol ODriveInterfacingBoard-rescue:LED-Device -> ODriveInterfacingBoard-rescue:LED-Device-ODriveInterfacingBoard-rescue
- U1: symbol ODriveInterfacingBoard-rescue:ODrive-ODrive -> ODriveInterfacingBoard-rescue:ODrive-ODrive-ODriveInterfacingBoard-rescue
Connections:
- net Rx: now also Conn9.1, R1.1; no longer Conn9.3, R2.1
- net Tx: now also Conn9.3, R2.1; no longer Conn9.1, R1.1

Commit message: Added Usb connectors in schematic
USB to USB to USB to USB!!!!
Parts:
- added J1: USB_B_Micro, symbol Connector:USB_B_Micro
- added J2: USB_A, symbol Connector:USB_A
- 50W2RJ1, R1, R10, R11, R12, R13, R14, R2, R3, R4, R5, R6, R7, R8, R9: symbol ODriveInterfacingBoard-rescue:R-Device-ODriveInterfacingBoard-rescue -> ODriveInterfacingBoard-rescue:R-Device-ODriveInterfacingBoard-rescue-ODriveInterfacingBoard-rescue
- Conn3, Conn7, Conn8: symbol ODriveInterfacingBoard-rescue:AndersonPP-MRDT_Connectors-ODriveInterfacingBoard-rescue -> ODriveInterfacingBoard-rescue:AndersonPP-MRDT_Connectors-ODriveInterfacingBoard-rescue-ODriveInterfacingBoard-rescue
- Conn9: symbol ODriveInterfacingBoard-rescue:Molex_SL_03-MRDT_Connectors-ODriveInterfacingBoard-rescue -> ODriveInterfacingBoard-rescue:Molex_SL_03-MRDT_Connectors-ODriveInterfacingBoard-rescue-ODriveInterfacingBoard-rescue
- D1, D10, D11, D12, D13, D14, D15, D16, D17, D18, D19, D2, D20, D3, D4, D5, D6, D7, D8, D9: symbol ODriveInterfacingBoard-rescue:LED-Device-ODriveInterfacingBoard-rescue -> ODriveInterfacingBoard-rescue:LED-Device-ODriveInterfacingBoard-rescue-ODriveInterfacingBoard-rescue
- U1: symbol ODriveInterfacingBoard-rescue:ODrive-ODrive-ODriveInterfacingBoard-rescue -> ODriveInterfacingBoard-rescue:ODrive-ODrive-ODriveInterfacingBoard-rescue-ODriveInterfacingBoard-rescue
Connections:
- net GND: now also J1.5 (GND), J2.4 (GND)
- new net: J1.6 (Shield), J2.5 (Shield)
- new net D+: J1.3 (D+), J2.3 (D+)
- new net D-: J1.2 (D-), J2.2 (D-)
- new net VBUS: J1.1 (VBUS), J2.1 (VBUS)

Commit message: Post - Review
Connections:
- no-connect marks 16 -> 17
Changed lines of the file:
@@
 $EndComp
-Wire Wire Line
-	8700 2050 8900 2050
-Wire Wire Line
-	8700 2250 8850 2250
 Wire Wire Line
 	8700 2350 9000 2350
@@
 	8300 2650 8300 2850
 $Comp
-L power:GND #PWR?
+L power:GND #PWR0105
 U 1 1 5F87E9A7
 P 8400 2800
-F 0 "#PWR?" H 8400 2550 50  0001 C CNN
+F 0 "#PWR0105" H 8400 2550 50  0001 C CNN
 F 1 "GND" H 8405 2627 50  0000 C CNN
 F 2 "" H 8400 2800 50  0001 C CNN
@@
 	1    0    0    -1
 $EndComp
-Text Label 8900 2050 0    50   ~ 0
-VBUS
-Text Label 8850 2250 0    50   ~ 0
-D+
-Text Label 9000 2350 0    50   ~ 0
-D-
-Wire Wire Line
-	8750 3450 9000 3450
-Wire Wire Line
-	8750 3650 9000 3650
 Wire Wire Line
 	8750 3750 9150 3750
@@
 Wire Wire Line
 	8100 2850 8300 2850
-Text Label 9000 3450 0    50   ~ 0
-VBUS
-Text Label 9000 3650 0    50   ~ 0
-D+
-Text Label 9150 3750 0    50   ~ 0
-D-
 $Comp
-L power:GND #PWR?
+L power:GND #PWR0106
 U 1 1 5F8ADC68
 P 8450 4200
-F 0 "#PWR?" H 8450 3950 50  0001 C CNN
+F 0 "#PWR0106" H 8450 3950 50  0001 C CNN
 F 1 "GND" H 8455 4027 50  0000 C CNN
 F 2 "" H 8450 4200 50  0001 C CNN
@@
 	1    0    0    -1
 $EndComp
+Text GLabel 8950 1950 0    50   Input ~ 0
+VBUS
+Text GLabel 8850 2150 0    50   Input ~ 0
+D+
+Text GLabel 8850 2450 0    50   Input ~ 0
+D-
+Wire Wire Line
+	8950 1950 8950 2050
+Wire Wire Line
+	8700 2050 8950 2050
+Wire Wire Line
+	8850 2150 8900 2150
+Wire Wire Line
+	8900 2150 8900 2250
+Wire Wire Line
+	8700 2250 8900 2250
+Wire Wire Line
+	9000 2350 9000 2450
+Wire Wire Line
+	9000 2450 8850 2450
+Text GLabel 9050 3350 0    50   Input ~ 0
+VBUS
+Text GLabel 9000 3550 0    50   Input ~ 0
+D+
+Text GLabel 9000 3850 0    50   Input ~ 0
+D-
+Wire Wire Line
+	9050 3350 9100 3350
+Wire Wire Line
+	9100 3350 9100 3450
+Wire Wire Line
+	8750 3450 9100 3450
+Wire Wire Line
+	9000 3550 9050 3550
+Wire Wire Line
+	9050 3550 9050 3650
+Wire Wire Line
+	8750 3650 9050 3650
+Wire Wire Line
+	9150 3750 9150 3850
+Wire Wire Line
+	9150 3850 9000 3850
+NoConn ~ 8750 3850
 $EndSCHEMATC
