File: ODriveInterfacingBoard/_autosave-ODriveInterfacingBoard.kicad_pcb (KiCad board)
At the start: 2 copper layers, 144.3 x 126.2 mm, 34 parts, among them U1 ODrive

Commit message: finished the via stitching. ready to make gerbs
Other:
- board text added: "ODRIVE INTERFACING BOARD, REV. 2 MARS ROVER DESIGN TEAM MISSOURI S&T, 2019 BRIAN DAHLMAN"
- board text removed: "ODRIVE INTERFACING BOARD, REV. 1 MARS ROVER DESIGN TEAM MISSOURI S&T, 2019 BRIAN DAHLMAN"
Changed lines of the file:
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@@
   (gr_line (start 179.324 52.07) (end 179.324 50.038) (layer Edge.Cuts) (width 0.15))
   (gr_line (start 35.052 53.086) (end 35.052 50.038) (layer Edge.Cuts) (width 0.15))
-  (gr_text "ODRIVE INTERFACING BOARD, REV. 1\nMARS ROVER DESIGN TEAM\nMISSOURI S&T, 2019\nBRIAN DAHLMAN" (at 99.06 160.02) (layer F.SilkS)
+  (gr_text "ODRIVE INTERFACING BOARD, REV. 2\nMARS ROVER DESIGN TEAM\nMISSOURI S&T, 2019\nBRIAN DAHLMAN" (at 99.06 160.02) (layer F.SilkS)
     (effects (font (size 1.5 1.5) (thickness 0.3)))
   )
