File: ODriveInterfacingBoard/_autosave-ODriveInterfacingBoard.kicad_pcb (KiCad board)
At the start: 2 copper layers, 32 parts, among them U1 ODrive

Commit message: blahblah I pushed
Parts:
- moved D1 125.1 mm to (31.0, 101.3)
- moved D11 125.1 mm to (31.0, 103.9)
- moved D13 125.1 mm to (31.0, 106.5)
- moved R6 125.1 mm to (30.9, 114.0)
- moved R8 125.1 mm to (30.9, 109.0)
- moved R9 125.1 mm to (30.9, 111.5)
- moved D14 78.7 mm to (13.7, 98.3)
- moved D10 78.7 mm to (9.34, 90.5)
- moved D12 78.7 mm to (18.1, 97.1)
- moved D2 78.7 mm to (13.7, 90.5)
- moved D3 78.7 mm to (9.34, 93.1)
- moved D4 78.7 mm to (9.34, 97.1)
- moved D5 78.7 mm to (13.7, 93.1)
- moved D6 78.7 mm to (18.1, 90.5)
- moved D7 78.7 mm to (18.1, 93.1)
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Other:
- board outline added: 177.9 x 50 mm
