File: ODriveInterfacingBoard_Reduced/ODriveInterfacingBoard.kicad_pcb (KiCad board)
At the start: 2 copper layers, 144.3 x 126.2 mm, 44 parts, among them U1 ODrive, U2 MAX3077E

Commit message: Created Gerbs
Connections:
- U2 pad 2: Tx -> Rx
- U2 pad 3: Rx -> Tx
Routing:
- net Rx: track 159.6 -> 163.8 mm
- net Tx: track 159.7 -> 158.5 mm, vias 3 -> 4
